File: Hardware/Teensy_Audio_Board_Test/Teensy_Audio_Board_Test.kicad_pcb (KiCad board)
At the start: 4 copper layers, 36.8 x 38.1 mm, 38 parts, among them J1 Conn_02x05_Odd_Even, J2 Micro_SD_Card_Det2, J3 AudioJack3, J4 Conn_01x14_Pin, J5 Conn_01x14_Pin

Commit message: Finalizing DRC Edits
Routing:
- net +3.3V: track 28.5 -> 47.9 mm, vias 15 -> 13
- net GND: track 27.0 -> 33.1 mm
Changed lines of the file:
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@@
 		(at 128.27 66.04 -90)
 		(property "Reference" "MK1"
-			(at 0 -2.286 -180)
+			(at 0 -2.286 180)
 			(layer "B.SilkS")
 			(effects
@@
 		(at 153.035 85.725 90)
 		(property "Reference" "R8"
-			(at 4.953 -2.667 -180)
+			(at 4.953 -2.667 180)
 			(layer "B.SilkS")
 			(effects
@@
 		(at 129.032 71.374 180)
 		(property "Reference" "U2"
-			(at -0.23 1.45 -0)
+			(at -0.23 1.45 0)
 			(layer "B.SilkS")
 			(effects
@@
 		(tags "capacitor")
 		(property "Reference" "C12"
-			(at -0.508 0 -0)
+			(at -0.508 0 0)
 			(layer "B.SilkS")
 			(effects
@@
 		(tags "QFN NoLead")
 		(property "Reference" "U1"
-			(at 0 2.032 -360)
+			(at 0 2.032 0)
 			(layer "B.SilkS")
 			(effects
@@
 		)
 		(property "Value" "~"
-			(at 0 3.8 360)
+			(at 0 3.8 0)
 			(layer "F.Fab")
 			(effects
@@
 		)
 		(property "Footprint" "Package_DFN_QFN:QFN-32-1EP_5x5mm_P0.5mm_EP3.6x3.6mm"
-			(at 0 0 360)
+			(at 0 0 0)
 			(layer "F.Fab")
 			(hide yes)
@@
 		)
 		(property "Datasheet" ""
-			(at 0 0 360)
+			(at 0 0 0)
 			(layer "F.Fab")
 			(hide yes)
@@
 		)
 		(property "Description" ""
-			(at 0 0 360)
+			(at 0 0 0)
 			(layer "F.Fab")
 			(hide yes)
@@
 		)
 		(fp_text user "${REFERENCE}"
-			(at 0 0 360)
+			(at 0 0 0)
 			(layer "F.Fab")
 			(effects
@@
 		(tags "3.5mm audio cui horizontal jack stereo")
 		(property "Reference" "J3"
-			(at 0 1.016 -180)
+			(at 0 1.016 180)
 			(layer "B.SilkS")
 			(effects
@@
 		(tags "capacitor")
 		(property "Reference" "C4"
-			(at 0 -0.762 -180)
+			(at 0 -0.762 180)
 			(layer "B.SilkS")
 			(effects
@@
 		(tags "Through hole pin header THT 2x05 2.54mm double row")
 		(property "Reference" "J1"
-			(at 4.064 -2.794 -180)
+			(at 4.064 -2.794 180)
 			(layer "B.SilkS")
 			(effects
@@
 		(tags "resistor")
 		(property "Reference" "R1"
-			(at 0 0 -0)
+			(at 0 0 0)
 			(layer "B.SilkS")
 			(effects
@@
 		(tags "capacitor")
 		(property "Reference" "C11"
-			(at 0 0 -0)
+			(at 0 0 0)
 			(layer "B.SilkS")
 			(effects
@@
 		(tags "resistor")
 		(property "Reference" "R2"
-			(at 0 0 -0)
+			(at 0 0 0)
 			(layer "B.SilkS")
 			(effects
@@
 		(tags "resistor")
 		(property "Reference" "R5"
-			(at 0 0 -0)
+			(at 0 0 0)
 			(layer "B.SilkS")
 			(effects
@@
 		(tags "resistor")
 		(property "Reference" "R6"
-			(at 0 0 -0)
+			(at 0 0 0)
 			(layer "B.SilkS")
 			(effects
@@
 		(tags "resistor")
 		(property "Reference" "R3"
-			(at -1.778 0.762 -0)
+			(at -1.778 0.762 0)
 			(layer "B.SilkS")
 			(effects
@@
 		(tags "capacitor")
 		(property "Reference" "C9"
-			(at 0 -0.254 -0)
+			(at 0 -0.254 0)
 			(layer "B.SilkS")
 			(effects
@@
 		(tags "capacitor")
 		(property "Reference" "C1"
-			(at 0 0 -0)
+			(at 0 0 0)
 			(layer "B.SilkS")
 			(effects
@@
 		(tags "capacitor")
 		(property "Reference" "C3"
-			(at 0 0 -0)
+			(at 0 0 0)
 			(layer "B.SilkS")
 			(effects
@@
 		(tags "capacitor")
 		(property "Reference" "C14"
-			(at 0 0 -0)
+			(at 0 0 0)
 			(layer "B.SilkS")
 			(effects
@@
 		(tags "resistor")
 		(property "Reference" "R7"
-			(at 0 0 -0)
+			(at 0 0 0)
 			(layer "B.SilkS")
 			(effects
@@
 		(tags "Through hole pin header THT 1x14 2.54mm single row")
 		(property "Reference" "J4"
-			(at 2.794 0.254 360)
+			(at 2.794 0.254 0)
 			(layer "B.SilkS")
 			(effects
@@
 		)
 		(fp_text user "${REFERENCE}"
-			(at 0 -16.51 360)
+			(at 0 -16.51 0)
 			(layer "B.Fab")
 			(effects
@@
 		(tags "Through hole pin header THT 1x14 2.54mm single row")
 		(property "Reference" "J5"
-			(at -2.032 0.508 360)
+			(at -2.032 0.508 0)
 			(layer "B.SilkS")
 			(effects
@@
 		)
 		(fp_text user "${REFERENCE}"
-			(at 0 -16.51 360)
+			(at 0 -16.51 0)
 			(layer "B.Fab")
 			(effects
@@
 	)
 	(via
-		(at 137.16 76.708)
-		(size 0.6)
-		(drill 0.3)
-		(layers "F.Cu" "B.Cu")
-		(free yes)
-		(net 1)
-	)
-	(via
 		(at 146.812 72.39)
 		(size 0.6)
@@
 	)
 	(via
-		(at 137.16 73.152)
-		(size 0.6)
-		(drill 0.3)
-		(layers "F.Cu" "B.Cu")
-		(free yes)
-		(net 1)
-	)
-	(via
 		(at 158.369 83.566)
 		(size 0.6)
@@
 	)
 	(segment
-		(start 137.16 73.152)
-		(end 137.16 76.708)
+		(start 144.718265 60.898265)
+		(end 145.542 61.722)
+		(width 0.254)
+		(layer "In2.Cu")
+		(net 1)
+	)
+	(segment
+		(start 158.912 73.465654)
+		(end 160.02 74.573654)
+		(width 0.2)
+		(layer "In2.Cu")
+		(net 1)
+	)
+	(segment
+		(start 133.35 59.69)
+		(end 134.558265 60.898265)
+		(width 0.254)
+		(layer "In2.Cu")
+		(net 1)
+	)
+	(segment
+		(start 159.512 67.564)
+		(end 158.912 68.164)
+		(width 0.2)
+		(layer "In2.Cu")
+		(net 1)
+	)
+	(segment
+		(start 158.912 68.164)
+		(end 158.912 73.465654)
+		(width 0.2)
+		(layer "In2.Cu")
+		(net 1)
+	)
+	(segment
+		(start 160.02 74.573654)
+		(end 160.02 76.454)
+		(width 0.2)
+		(layer "In2.Cu")
+		(net 1)
+	)
+	(segment
+		(start 134.558265 60.898265)
+		(end 144.718265 60.898265)
+		(width 0.254)
+		(layer "In2.Cu")
+		(net 1)
+	)
+	(segment
+		(start 160.02 76.454)
+		(end 160.274 76.708)
 		(width 0.2)
 		(layer "In2.Cu")
@@
 	)
 	(segment
+		(start 143.39 54.49)
+		(end 142.24 53.34)
+		(width 0.2)
+		(layer "In1.Cu")
+		(net 2)
+	)
+	(segment
+		(start 147.32 55.88)
+		(end 145.93 54.49)
+		(width 0.2)
+		(layer "In1.Cu")
+		(net 2)
+	)
+	(segment
+		(start 145.93 54.49)
+		(end 143.39 54.49)
+		(width 0.2)
+		(layer "In1.Cu")
+		(net 2)
+	)
+	(segment
 		(start 157.099 83.566)
 		(end 157.099 85.259)
@@
 		(polygon
 			(pts
-				(xy 126.492 50.292) (xy 163.068 50.292) (xy 163.068 88.138) (xy 126.492 88.138)
+				(xy 126.492 59.69) (xy 163.068 59.69) (xy 163.068 88.138) (xy 126.492 88.138)
 			)
 		)
