File: Hardware/Teensy_Audio_Board_Test/Teensy_Audio_Board_Test.kicad_sch (KiCad schematic)
At the start: 38 parts, among them J1 Conn_02x05_Odd_Even, J2 Micro_SD_Card_Det2, J3 AudioJack3, J4 Conn_01x14_Pin, J5 Conn_01x14_Pin

Commit message: Finalizing DRC Edits
Other:
- note removed: "Wires for MCLK, BCLK, LRCLK, TX, and RX should be kept short"
Changed lines of the file:
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@@
-		)
-	)
-	(text "Wires for MCLK, BCLK, LRCLK, TX, and RX should be kept short"
-		(exclude_from_sim no)
-		(at 134.366 7.366 0)
-		(effects
-			(font
-				(size 1.27 1.27)
-			)
 		)
 	)
